Commit message: Updated to Ranger2
While here, catkinize the package. Successfully tested with Indigo

File: urdf/ranger.urdf (robot description, URDF)
Before this commit: robot ranger, 7 links, 6 joints
Links:
- link box: geometry visual mesh filename=package://ranger_description/urdf/meshes/ranger.dae
- link l_eye_link: geometry 
- link l_wheel_link: geometry 
- link r_eye_link: geometry 
- link r_wheel_link: geometry 
Joints:
- joint base_link_box_joint: origin xyz=-0.13 0.0 0.0 rpy=0 0.0 0.0 -> xyz=0.0 0.0 0.0 rpy=0 0.0 0.0
- joint base_link_l_wheel_joint: origin xyz=0.0 -0.205 -0.011 rpy=1.52 0.0 0.0 -> xyz=0.0 -0.16 0.053 rpy=1.52 0.0 0.0
- joint base_link_r_wheel_joint: origin xyz=0.0 0.205 -0.011 rpy=-1.52 0.0 0.0 -> xyz=0.0 0.16 0.053 rpy=-1.52 0.0 0.0

Commit message: Added links for the IR sensors and adjusted RGB/depth frames

File: urdf/ranger.urdf (robot description, URDF)
Before this commit: robot ranger, 7 links, 6 joints
Links:
- added link ir_center
- added link ir_left
- added link ir_right
- added link rgb_camera_link
Joints:
- added joint base_link_ir_center_joint: type fixed, parent base_link, child ir_center, origin xyz=0.08 0.0 0.073 rpy=0.0 0.0 0.0
- added joint base_link_ir_left_joint: type fixed, parent base_link, child ir_left, origin xyz=0.08 0.115 0.073 rpy=0.0 0.0 0.0
- added joint base_link_ir_right_joint: type fixed, parent base_link, child ir_right, origin xyz=0.08 -0.115 0.073 rpy=0.0 0.0 0.0
- added joint base_link_rgb_camera_joint: type fixed, parent base_link, child rgb_camera_link, origin xyz=0.055 0.024 0.36 rpy=0 0.0 0.0
- joint base_link_depth_camera_joint: origin xyz=0.055 0.0 0.317 rpy=0 0.0 0.0 -> xyz=0.055 0.051 0.36 rpy=0 0.0 0.0

Commit message: added camera link to robot description

File: urdf/ranger.urdf (robot description, URDF)
Before this commit: robot ranger, 11 links, 10 joints
Links:
- added link camera_link
Joints:
- added joint base_link_camera_joint: type fixed, parent base_link, child camera_link, origin xyz=0.055 0.0 0.36 rpy=0 0.0 0.0
- joint base_link_depth_camera_joint: origin xyz=0.055 0.051 0.36 rpy=0 0.0 0.0 -> xyz=0.055 0.050 0.36 rpy=0 0.0 0.0
